File: FORWARD-MAIN/_autosave-FORWARD-PCB.kicad_sch (KiCad schematic)
At the start: 43 parts, among them J1 USB_B_Micro, J2 Conn_01x03_Socket, J3 Conn_01x13_Socket, J4 Conn_01x08_Socket, Q1 SS8050-G, Q2 SS8050-G, U2 CP2102N-Axx-xQFN28, U5 ESP32-WROOM-32D

Commit message: itried
Connections:
- net LIGHT-IO4-26: now also U5.26 (IO4); no longer U5.29 (IO5)
- net Wheels-IO16-27: now also J3.10 (Pin_10), U5.29 (IO5); no longer J3.11 (Pin_11), U5.26 (IO4)
- net Wheels-IO17-28: now also J3.11 (Pin_11); no longer J3.12 (Pin_12)
- net Wheels-IO5-29: now also J3.12 (Pin_12); no longer J3.10 (Pin_10)
Changed lines of the file:
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@@
-		)
-	)
-	(label "Wheels-IO16-27"
-		(at 254 66.04 0)
-		(effects
-			(font
-				(size 1.27 1.27)
-			)
-			(justify left bottom)
 		)
 	)
@@
 		)
 	)
-	(label "Wheels-IO17-28"
-		(at 142.24 175.26 180)
-		(effects
-			(font
-				(size 1.27 1.27)
-			)
-			(justify right bottom)
-		)
-	)
 	(label "Haptics-IO32"
 		(at 142.24 154.94 180)
@@
 		)
 	)
-	(label "LIGHT-IO4-26"
-		(at 254 68.58 0)
-		(effects
-			(font
-				(size 1.27 1.27)
-			)
-			(justify left bottom)
-		)
-	)
 	(label "USB_DN"
 		(at 110.49 72.39 0)
@@
 		)
 	)
+	(label "Wheels-IO16-27"
+		(at 254 68.58 0)
+		(effects
+			(font
+				(size 1.27 1.27)
+			)
+			(justify left bottom)
+		)
+	)
 	(label "Haptics-IO26"
 		(at 142.24 149.86 180)
@@
 		)
 	)
+	(label "LIGHT-IO4-26"
+		(at 254 66.04 0)
+		(effects
+			(font
+				(size 1.27 1.27)
+			)
+			(justify left bottom)
+		)
+	)
 	(label "RXD0"
 		(at 254 63.5 0)
@@
 		)
 	)
+	(label "Wheels-IO16-27"
+		(at 142.24 170.18 180)
+		(effects
+			(font
+				(size 1.27 1.27)
+			)
+			(justify right bottom)
+		)
+	)
 	(label "TXD"
 		(at 187.96 62.23 180)
@@
 		)
 	)
-	(label "Wheels-IO16-27"
-		(at 142.24 172.72 180)
-		(effects
-			(font
-				(size 1.27 1.27)
-			)
-			(justify right bottom)
-		)
-	)
 	(label "Haptics-IO27"
 		(at 142.24 152.4 180)
@@
 		)
 	)
-	(label "Wheels-IO5-29"
-		(at 142.24 170.18 180)
-		(effects
-			(font
-				(size 1.27 1.27)
-			)
-			(justify right bottom)
-		)
-	)
 	(label "EN"
 		(at 110.49 120.65 0)
@@
 		)
 	)
+	(label "Wheels-IO17-28"
+		(at 142.24 172.72 180)
+		(effects
+			(font
+				(size 1.27 1.27)
+			)
+			(justify right bottom)
+		)
+	)
 	(label "TRIG_3"
 		(at 254 91.44 0)
@@
 		)
 	)
+	(label "Wheels-IO5-29"
+		(at 142.24 175.26 180)
+		(effects
+			(font
+				(size 1.27 1.27)
+			)
+			(justify right bottom)
+		)
+	)
