File: FORWARD-MAIN/FORWARD-PCB.kicad_pcb (KiCad board)
At the start: 2 copper layers, 96.3 x 67.5 mm, 46 parts, among them J1 USB_B_Micro, J2 Conn_01x03_Socket, J5 Conn_01x14_Pin, Q1 SS8050-G, Q2 SS8050-G, U1 BNO055, U2 CP2102N-Axx-xQFN28, U5 ESP32-WROOM-32D

Commit message: Redesign of pcb
Parts:
- removed D1: BAT760-7, pcb-footprints:SOD2513X120N
- removed D2, D3, D5: LESD5D5.0CT1G, pcb-footprints:TVS_LESD5D5.0CT1G
- removed J5: Conn_01x14_Pin, Connector_PinHeader_2.54mm:PinHeader_1x14_P2.54mm_Horizontal
- removed Q1, Q2: SS8050-G, pcb-footprints:TRANS_SS8050-G
- removed U1: BNO055, Package_LGA:LGA-28_5.2x3.8mm_P0.5mm
- added J3: Conn_01x16_Socket, Connector_Phoenix_MC:PhoenixContact_MC_1,5_16-G-3.81_1x16_P3.81mm_Horizontal, F.Cu at (93.2, 156.3)
- added J4: Conn_01x08_Socket, Connector_PinSocket_2.54mm:PinSocket_1x08_P2.54mm_Vertical, F.Cu at (112.3, 146.0)
- added TP4: TestPoint, TestPoint:TestPoint_Loop_D2.50mm_Drill1.0mm_LowProfile, F.Cu at (140.3, 139.8)
- moved S2 93.2 mm to (170.1, 157.3), turned to 180 degrees
- moved J2 82.5 mm to (114.8, 103.3), turned to 180 degrees
- moved Boot1 65.4 mm to (96.8, 101.8)
- moved R3 64.8 mm to (160.8, 149.7), turned to 90 degrees
- moved R4 60.2 mm to (160.3, 145.3), turned to 90 degrees
- moved R18 55.9 mm to (134.3, 109.2), turned to -90 degrees
- moved Reset1 52.0 mm to (96.8, 109.8)
- moved J1 48.8 mm to (184.4, 126.5), turned to 90 degrees
- moved R11 48.8 mm to (171.8, 133.4), turned to 90 degrees
- moved C10 47.3 mm to (130.3, 106.3), turned to 180 degrees
- moved R12 43.9 mm to (176.8, 131.2), turned to -90 degrees
- moved R14 40.9 mm to (167.8, 133.3), turned to 90 degrees
- moved L1 38.5 mm to (97.2, 136.3), turned to -90 degrees
- moved U2 36.3 mm to (169.3, 125.8)
- moved C9 32.8 mm to (151.2, 140.8)
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Connections:
- C1 pad 1: /IO0 -> /RST
- Reset1 pad 2: /IO0 -> /RST
- U5 pad 10: /TRIG_3 -> /Haptics-IO25
- U5 pad 11: /TRIG_4 -> /Haptics-IO26
- U5 pad 12: /Wheels-IO27 -> /Haptics-IO27
- U5 pad 13: /Haptics-IO14 -> /SDA
- U5 pad 14: /Haptics-IO12 -> /SCL
- U5 pad 16: /Haptics-IO13 -> /P0W
- U5 pad 23: /P0W -> /ECHO_2
- U5 pad 24: /Haptics-IO2 -> /TRIG_2
- U5 pad 25: /IO0 -> /Wheels-IO0
- U5 pad 26: /Haptics-IO4 -> /Wheels-IO4
- U5 pad 29: /Haptics-IO5 -> /Wheels-IO5
- U5 pad 31: /Wheels-IO19 -> /ECHO_3
- U5 pad 33: /SDA -> /TRIG_3
- U5 pad 36: /SCL -> /ECHO_4
- U5 pad 37: /Wheels-IO23 -> /TRIG_4
- U5 pad 38: /ECHO_1 -> GND
- U5 pad 39: /ECHO_2 -> GND
- U5 pad 4: unconnected-(U5-SENSOR_VP-Pad4) -> /RST
- U5 pad 5: unconnected-(U5-SENSOR_VN-Pad5) -> /ECHO_1
- U5 pad 6: /ECHO_3 -> /TRIG_1
- U5 pad 7: /ECHO_4 -> /Haptics-IO35
- U5 pad 8: /TRIG_1 -> /Haptics-IO32
- U5 pad 9: /TRIG_2 -> /Haptics-IO33
Routing:
- net +5V: track 0.00 -> 195.8 mm
- net +3.3V: track 0.00 -> 163.0 mm, vias 0 -> 1
- net /Wheels-IO5: track 0.00 -> 74.9 mm, vias 0 -> 2
- net /Haptics-IO25: track 0.00 -> 72.0 mm, vias 0 -> 2
- net /Haptics-IO26: track 0.00 -> 71.9 mm, vias 0 -> 1
- net /Haptics-IO32: track 0.00 -> 68.5 mm, vias 0 -> 1
- net /Haptics-IO27: track 0.00 -> 67.9 mm, vias 0 -> 1
- net /Haptics-IO33: track 0.00 -> 64.9 mm, vias 0 -> 1
- net /Wheels-IO0: track 0.00 -> 62.4 mm, vias 0 -> 1
- net /Wheels-IO4: track 0.00 -> 61.2 mm, vias 0 -> 2
- net /SCL: track 0.00 -> 57.9 mm, vias 0 -> 1
- net /Wheels-IO18: track 0.00 -> 57.7 mm, vias 0 -> 1
- net /Haptics-IO35: track 0.00 -> 57.6 mm, vias 0 -> 1
- net /Wheels-IO16: track 0.00 -> 56.7 mm, vias 0 -> 1
- net /SDA: track 0.00 -> 56.6 mm
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- added copper zone on B.Cu, net GND
Other:
- copper layers 2 -> 4

Commit message: itried
Parts:
- removed R3: 1k, Resistor_SMD:R_0805_2012Metric
- removed R4: 2k, Resistor_SMD:R_0805_2012Metric
- removed S2: Conn_01x04_Socket, Connector_JST:JST_EH_S4B-EH_1x04_P2.50mm_Horizontal
- added D1: BAT760-7, footprints:SOD2513X120N, F.Cu at (119.2, 94.4)
- added D2: LESD5D5.0CT1G, footprints:TVS_LESD5D5.0CT1G, F.Cu at (121.2, 121.8)
- added D3: LESD5D5.0CT1G, footprints:TVS_LESD5D5.0CT1G, F.Cu at (123.7, 102.6)
- added D5: LESD5D5.0CT1G, footprints:TVS_LESD5D5.0CT1G, F.Cu at (134.2, 120.8)
- added Q1: SS8050-G, footprints:TRANS_SS8050-G, F.Cu at (139.5, 101.8)
- added Q2: SS8050-G, footprints:TRANS_SS8050-G, F.Cu at (139.5, 96.8)
- J2: footprint Connector_JST:JST_PH_S3B-PH-K_1x03_P2.00mm_Horizontal -> Connector_PinHeader_2.54mm:PinHeader_1x03_P2.54mm_Horizontal
- J3: value Conn_01x16_Socket -> Conn_01x13_Socket; footprint Connector_Phoenix_MC:PhoenixContact_MC_1,5_16-G-3.81_1x16_P3.81mm_Horizontal -> Connector_Phoenix_MC:PhoenixContact_MC_1,5_13-G-3.81_1x13_P3.81mm_Horizontal
- TP4: footprint TestPoint:TestPoint_Loop_D2.50mm_Drill1.0mm_LowProfile -> TestPoint:TestPoint_Pad_1.0x1.0mm
- moved G*** 132.2 mm to (69.6, 85.1)
- moved L1 81.2 mm to (105.0, 55.5), turned to 180 degrees
- moved S1 78.2 mm to (67.5, 55.5), turned to 0 degrees
- moved R1 69.4 mm to (72.9, 61.0)
- moved Boot1 67.8 mm to (150.0, 143.9), turned to 90 degrees
- moved R2 66.5 mm to (74.4, 66.6), turned to -90 degrees
- moved C9 65.5 mm to (88.5, 121.8)
- moved R13 63.2 mm to (102.7, 119.3), turned to 0 degrees
- moved R16 62.9 mm to (149.0, 60.0), turned to 0 degrees
- moved R5 61.7 mm to (157.5, 82.5), turned to 180 degrees
- moved S3 59.4 mm to (165.0, 79.8)
- moved R17 57.7 mm to (153.0, 63.0), turned to 0 degrees
- moved R15 57.4 mm to (89.0, 95.8), turned to 180 degrees
- moved R12 56.0 mm to (132.7, 96.8), turned to 0 degrees
- moved R6 55.8 mm to (156.5, 87.6), turned to -90 degrees
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Connections:
- net /Wheels-IO16 renamed /Wheels-IO17-28
- net /Wheels-IO17 renamed /Wheels-IO5-29
- net /Wheels-IO18 renamed /Wheels-IO18-30
- net /Wheels-IO4 renamed /LIGHT-IO4-26
- net /Wheels-IO5 renamed /Wheels-IO16-27
- J3 pad 1: +5V -> /Haptics-IO25
- J3 pad 2: /Haptics-IO25 -> /Haptics-IO26
- J3 pad 3: /Haptics-IO26 -> /Haptics-IO27
- J3 pad 4: /Haptics-IO27 -> /Haptics-IO32
- J3 pad 5: /Haptics-IO32 -> /Haptics-IO33
- J3 pad 6: /Haptics-IO33 -> /Haptics-IO35
- J3 pad 7: /Haptics-IO35 -> /P0W-IO13-16
- J3 pad 8: /Wheels-IO0 -> /PHOTO-IO2-24
- R14 pad 1: Net-(U2-~{RST}) -> /RST
- U2 pad 9: Net-(U2-~{RST}) -> /RST
- U5 pad 10: /Haptics-IO25 -> /Haptics-IO32
- U5 pad 11: /Haptics-IO26 -> /Haptics-IO33
- U5 pad 12: /Haptics-IO27 -> /Haptics-IO35
- U5 pad 16: /P0W -> /P0W-IO13-16
- U5 pad 23: /ECHO_2 -> /ECHO_1
- U5 pad 24: /TRIG_2 -> /PHOTO-IO2-24
- U5 pad 25: /Wheels-IO0 -> /IO0
- U5 pad 4: /RST -> unconnected-(U5-SENSOR_VP-Pad4)
- U5 pad 5: /ECHO_1 -> unconnected-(U5-SENSOR_VN-Pad5)
- U5 pad 7: /Haptics-IO35 -> /Haptics-IO25
- U5 pad 8: /Haptics-IO32 -> /Haptics-IO26
- U5 pad 9: /Haptics-IO33 -> /Haptics-IO27
Routing:
- net +5V: track 195.8 -> 0.00 mm
- net +3.3V: track 163.0 -> 0.00 mm, vias 1 -> 0
- net /P0W-IO13-16: track 0.00 -> 123.2 mm, vias 0 -> 2
- net /Wheels-IO16-27: track 74.9 -> 0.00 mm, vias 2 -> 0
- net /Wheels-IO0: track 62.4 -> 0.00 mm, vias 1 -> 0
- net /LIGHT-IO4-26: track 61.2 -> 0.00 mm, vias 2 -> 0
- net /Haptics-IO35: track 57.6 -> 116.5 mm, vias 1 -> 0
- net /SCL: track 57.9 -> 0.00 mm, vias 1 -> 0
- net /Wheels-IO18-30: track 57.7 -> 0.00 mm, vias 1 -> 0
- net /Wheels-IO17-28: track 56.7 -> 0.00 mm, vias 1 -> 0
- net /SDA: track 56.6 -> 0.00 mm
- net /Wheels-IO5-29: track 54.7 -> 0.00 mm, vias 1 -> 0
- net /Haptics-IO33: track 64.9 -> 117.3 mm, vias 1 -> 0
- net /Haptics-IO27: track 67.9 -> 120.3 mm, vias 1 -> 0
- net /Haptics-IO25: track 72.0 -> 123.7 mm, vias 2 -> 0
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- added copper zone on In1.Cu, net GND
- removed copper zone on B.Cu, net GND
Other:
- board size 96.3 x 67.5 mm -> 111.5 x 101.5 mm

Commit message: a good iteration!
Parts:
- added R3: 1k, Resistor_SMD:R_0805_2012Metric, F.Cu at (103.2, 66.4)
- added R4: 2k, Resistor_SMD:R_0805_2012Metric, F.Cu at (106.7, 68.9)
- added S2: Conn_01x04_Socket, Connector_JST:JST_EH_S4B-EH_1x04_P2.50mm_Horizontal, F.Cu at (96.8, 75.0)
- moved G*** 77.3 mm to (130.6, 132.4), turned to 90 degrees
- moved C8 73.3 mm to (151.0, 77.5)
- moved C9 71.8 mm to (145.0, 77.5), turned to 180 degrees
- moved D2 51.8 mm to (161.0, 155.0), turned to -90 degrees
- moved TP4 44.1 mm to (150.0, 100.5)
- moved R13 43.9 mm to (146.5, 122.5), turned to 90 degrees
- moved R16 42.6 mm to (191.5, 57.5)
- moved R17 42.6 mm to (195.5, 60.5)
- moved R10 38.5 mm to (167.5, 103.0)
- moved S3 37.9 mm to (196.0, 101.5)
- moved S4 37.9 mm to (196.0, 86.5)
- moved R9 35.9 mm to (163.0, 110.5)
- moved J3 35.0 mm to (98.6, 154.5)
- moved C1 34.7 mm to (142.4, 131.5), turned to 180 degrees
- moved Reset1 33.9 mm to (156.5, 156.4)
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Connections:
- net /Haptics-IO25 renamed /Haptics-IN1
- net /Haptics-IO26 renamed /Haptics-IN2
- net /Haptics-IO27 renamed /Haptics-IN3
- net /Haptics-IO32 renamed /Haptics-IN4
- net /Haptics-IO33 renamed /Haptics-ENA_PWM
- net /Haptics-IO35 renamed /Haptics-ENB_PWM
- net /Wheels-IO18-30 renamed /IO18-30
- J3 pad 10: /Wheels-IO16-27 -> /Wheels-RPWM
- J3 pad 11: /Wheels-IO17-28 -> /Wheels_LPWM
- J3 pad 12: /Wheels-IO5-29 -> /IO16-27
- U5 pad 23: /ECHO_1 -> /TRIG_2
- U5 pad 27: /Wheels-IO17-28 -> /Wheels-RPWM
- U5 pad 28: /Wheels-IO5-29 -> /Wheels_LPWM
- U5 pad 29: /Wheels-IO16-27 -> /IO16-27
- U5 pad 4: unconnected-(U5-SENSOR_VP-Pad4) -> /ECHO_1
- U5 pad 5: unconnected-(U5-SENSOR_VN-Pad5) -> /ECHO_2
Routing:
- net /IO18-30: track 0.00 -> 136.6 mm
- net /IO16-27: track 0.00 -> 134.6 mm
- net /Wheels_LPWM: track 0.00 -> 133.2 mm
- net /Wheels-RPWM: track 0.00 -> 131.4 mm
- net /LIGHT-IO4-26: track 0.00 -> 130.1 mm
- net /PHOTO-IO2-24: track 0.00 -> 127.6 mm
- net /SCL: track 0.00 -> 117.0 mm, vias 0 -> 2
- net /EN: track 0.00 -> 114.6 mm, vias 0 -> 4
- net /SDA: track 0.00 -> 96.3 mm, vias 0 -> 2
- net /TXD: track 0.00 -> 83.6 mm, vias 0 -> 2
- net /TRIG_2: track 0.00 -> 81.5 mm, vias 0 -> 1
- net /RXD: track 0.00 -> 80.5 mm, vias 0 -> 2
- net /VBUS: track 0.00 -> 66.9 mm, vias 0 -> 2
- net /USB_DP: track 0.00 -> 60.3 mm, vias 0 -> 2
- net /ECHO_2: track 0.00 -> 55.7 mm, vias 0 -> 2
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Other:
- board size 111.5 x 101.5 mm -> 107 x 114 mm
- board text added: "FORWARD Main Designers: Tobiah Bower Matthew Morello"

Commit message: ready to order (i think)
Parts:
- removed J2: Conn_01x03_Socket, Connector_PinHeader_2.54mm:PinHeader_1x03_P2.54mm_Horizontal
- added C4: 0.1uF, Capacitor_SMD:C_0805_2012Metric, F.Cu at (149.0, 86.5)
- added D4: LED, LED_SMD:LED_0805_2012Metric, F.Cu at (174.2, 101.2)
- added J5: Screw_Terminal_01x03, TerminalBlock_Phoenix:TerminalBlock_Phoenix_MPT-0,5-3-2.54_1x03_P2.54mm_Horizontal, F.Cu at (106.5, 110.0)
- added R20: 10k, Resistor_SMD:R_0805_2012Metric, F.Cu at (153.8, 86.8)
- L1: footprint Connector_JST:JST_PH_S6B-PH-K_1x06_P2.00mm_Horizontal -> Connector_JST:JST_EH_S6B-EH_1x06_P2.50mm_Horizontal
- moved G*** 97.8 mm to (193.1, 57.1), turned to 0 degrees
- moved R16 35.5 mm to (169.0, 85.0), turned to -90 degrees
- moved R17 30.8 mm to (172.5, 81.0), turned to -90 degrees
- moved D2 20.0 mm to (173.2, 139.2)
- moved J1 20.0 mm to (179.9, 142.8)
- moved Boot1 18.9 mm to (190.8, 141.2), turned to 0 degrees
- moved J3 17.6 mm to (106.0, 138.5)
- moved Reset1 17.1 mm to (164.5, 141.2), turned to 0 degrees
- moved D1 14.2 mm to (143.8, 87.5)
- moved R4 13.8 mm to (117.1, 78.1)
- moved R3 13.3 mm to (112.0, 76.5), turned to 0 degrees
- moved R14 9.56 mm to (147.6, 122.0)
- moved R11 9.53 mm to (153.8, 122.0)
- moved S2 8.80 mm to (105.5, 76.0)
- moved C2 8.58 mm to (173.0, 120.5)
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Connections:
- net /IO16-27 renamed /Wheel_R_LPWM
- net /IO18-30 renamed /Wheel_R_RPWM
- net /Wheels-RPWM renamed /Wheel_L_LPWM
- net /Wheels_LPWM renamed /Wheel_L_RPWM
- C1 pad 1: /RST -> /IO0
- C3 pad 1: +3.3V -> +5V
- C5 pad 1: +3.3V -> +5V
- R14 pad 1: /RST -> Net-(U2-~{RST})
- R14 pad 2: +3.3V -> +5V
- Reset1 pad 2: /RST -> /IO0
- U2 pad 6: +3.3V -> +5V
- U2 pad 7: +3.3V -> +5V
- U2 pad 9: /RST -> Net-(U2-~{RST})
- U5 pad 15: unconnected-(U5-GND-Pad15) -> GND
- U5 pad 25: /IO0 -> Net-(D4-K)
Routing:
- net +5V: track 0.00 -> 280.8 mm, vias 0 -> 6
- net GND: track 0.00 -> 105.9 mm, vias 0 -> 21
- net /IO0: track 36.8 -> 140.5 mm
- net /RXD: track 80.5 -> 37.4 mm
- net /RST: track 41.5 -> 0.00 mm, vias 2 -> 0
- net /TXD: track 83.6 -> 42.9 mm
- net Net-(D4-K): track 0.00 -> 28.5 mm, vias 0 -> 2
- net +3.3V: track 0.00 -> 20.7 mm, vias 0 -> 7
- net /Wheel_R_RPWM: track 136.6 -> 116.4 mm
- net /Haptics-IN4: track 116.7 -> 97.6 mm
- net /Haptics-IN3: track 120.5 -> 101.5 mm
- net /Haptics-IN1: track 128.0 -> 108.9 mm
- net /Haptics-IN2: track 124.4 -> 105.3 mm
- net /Haptics-ENA_PWM: track 112.5 -> 93.4 mm
- net /Haptics-ENB_PWM: track 108.1 -> 89.0 mm
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- added copper zone on In2.Cu, net +3.3V
Other:
- board size 107 x 114 mm -> 98 x 97.5 mm
- board text removed: "FORWARD Main Designers: Tobiah Bower Matthew Morello"
