File: FORWARD-MAIN/FORWARD-PCB.kicad_pcb (KiCad board)
At the start: 4 copper layers, 98 x 97.5 mm, 51 parts, among them J1 USB_B_Micro, J3 Conn_01x13_Socket, J4 Conn_01x08_Socket, J5 Screw_Terminal_01x03, Q1 SS8050-G, Q2 SS8050-G, U2 CP2102N-Axx-xQFN28, U5 ESP32-WROOM-32D

Commit message: PCB order rev 1.0
Parts:
- removed R15, R19: 3.2k, Resistor_SMD:R_0805_2012Metric
- removed TP4: TestPoint, Connector_PinHeader_2.54mm:PinHeader_1x01_P2.54mm_Vertical
- added J2: Conn_01x14_Socket, Connector_PinSocket_2.54mm:PinSocket_1x14_P2.54mm_Horizontal, F.Cu at (129.1, 136.3)
- added J6: Conn_01x02_Pin, Connector_PinSocket_2.54mm:PinSocket_1x02_P2.54mm_Vertical, F.Cu at (107.5, 87.5)
- Boot1, Reset1: footprint Button_Switch_SMD:SW_Tactile_SPST_NO_Straight_CK_PTS636Sx25SMTRLFS -> Button_Switch_SMD:SW_SPST_TL3305A
- D6: value LED -> Power-LED
- J3: value Conn_01x13_Socket -> Conn_01x02_Pin; footprint Connector_Phoenix_MSTB:PhoenixContact_MSTBA_2,5_13-G_1x13_P5.00mm_Horizontal -> Connector_PinSocket_2.54mm:PinSocket_1x02_P2.54mm_Vertical
- J5: footprint TerminalBlock_MetzConnect:TerminalBlock_MetzConnect_Type086_RT03403HBLC_1x03_P3.81mm_Horizontal -> TerminalBlock_Phoenix:TerminalBlock_Phoenix_MPT-0,5-3-2.54_1x03_P2.54mm_Horizontal
- R12: value 22.1k -> 1k
- R13: value 47.5k -> 1k
- R14: value 2k -> 10k
- moved G*** 108.4 mm to (117.9, 135.2), turned to 90 degrees
- moved J3 41.0 mm to (107.5, 97.5), turned to 90 degrees
- moved R13 30.3 mm to (115.5, 113.5), turned to -90 degrees
- moved R12 20.9 mm to (174.5, 103.5), turned to 90 degrees
- moved C3 9.92 mm to (138.5, 117.0), turned to -90 degrees
- moved C5 6.45 mm to (147.0, 114.5), turned to -90 degrees
- moved D3 5.02 mm to (142.5, 108.0)
- moved D2 3.00 mm to (170.2, 139.2)
- moved D4 2.15 mm to (173.0, 99.5), turned to 90 degrees
- moved R14 2.09 mm to (145.5, 122.0), turned to 180 degrees
- moved C1 1.50 mm to (142.8, 125.0)
- moved J5 1.26 mm to (106.1, 107.0)
- moved S4 0.90 mm to (194.0, 86.8)
- moved Reset1 0.55 mm to (193.8, 129.8)
- moved Boot1 0.50 mm to (190.8, 140.8), turned to 90 degrees
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Connections:
- C3 pad 1: +5V -> Net-(U2-VDD)
- C5 pad 1: +5V -> Net-(U2-VDD)
- D4 pad 2: /IO0 -> /LIGHT-IO4-26
- D6 pad 1: GND -> Net-(D6-K)
- J3 pad 1: /Haptics-IN1 -> /SDA
- J3 pad 2: /Haptics-IN2 -> /SCL
- R12 pad 1: /VBUS -> GND
- R12 pad 2: Net-(U2-VBUS) -> Net-(D4-K)
- R13 pad 1: GND -> Net-(D6-K)
- R13 pad 2: Net-(U2-VBUS) -> GND
- R14 pad 2: +5V -> Net-(U2-VDD)
- U2 pad 6: +5V -> Net-(U2-VDD)
- U2 pad 8: Net-(U2-VBUS) -> +5V
- U5 pad 24: /PHOTO-IO2-24 -> /LIGHT-IO4-26
- U5 pad 25: Net-(D4-K) -> /IO0
- U5 pad 26: /LIGHT-IO4-26 -> /PHOTO-IO2-24
Routing:
- net Net-(U2-VBUS): track 38.8 -> 0.00 mm
- net Net-(U2-VDD): track 0.00 -> 29.6 mm
- net /IO0: track 124.3 -> 152.4 mm, vias 2 -> 4
- net Net-(D4-K): track 28.5 -> 2.77 mm, vias 2 -> 0
- net /USB_DP: track 96.7 -> 117.3 mm
- net GND: track 109.2 -> 123.4 mm, vias 21 -> 20
- net /USB_DN: track 62.6 -> 70.9 mm
- net /PHOTO-IO2-24: track 103.4 -> 110.7 mm, vias 0 -> 2
- net /VBUS: track 82.0 -> 76.2 mm
- net /LIGHT-IO4-26: track 100.0 -> 105.8 mm, vias 0 -> 4
- net /EN: track 122.1 -> 127.9 mm
- net +3.3V: track 20.7 -> 15.1 mm, vias 7 -> 5
- net /SDA: track 94.8 -> 100.0 mm, vias 2 -> 1
- net /Wheel_R_RPWM: track 99.9 -> 104.8 mm
- net +5V: track 275.2 -> 270.5 mm, vias 5 -> 3
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Other:
- board size 98 x 97.5 mm -> 98 x 98 mm
- board text added: "Feedback Oriented Routing & Walker Assistance w/ Responsive Direction Designed by Tobiah Bower"

Commit message: MAIN PCB rev 2.0
Parts:
- J1: footprint Connector_USB:USB_Micro-B_Molex-105133-0031 -> Connector_USB:USB_Micro-B_Wuerth_629105150521
- moved G*** 6.64 mm to (111.7, 132.8), turned to 0 degrees
- moved J1 0.48 mm to (180.4, 142.7)
Routing:
- net /USB_DP: track 117.3 -> 112.0 mm
- net /USB_DN: track 70.9 -> 66.6 mm
- net GND: track 123.4 -> 124.5 mm
- net /VBUS: track 76.2 -> 75.5 mm
Other:
- board text removed: "Feedback Oriented Routing & Walker Assistance w/ Responsive Direction Designed by Tobiah Bower"

Commit message: fix i2c but still an issue
Parts:
- J2: value Conn_01x14_Socket -> Conn_01x15_Socket; footprint Connector_PinSocket_2.54mm:PinSocket_1x14_P2.54mm_Horizontal -> Connector_PinSocket_2.54mm:PinSocket_1x15_P2.54mm_Horizontal
- J5: value Screw_Terminal_01x03 -> Conn_01x03_Socket; footprint TerminalBlock_Phoenix:TerminalBlock_Phoenix_MPT-0,5-3-2.54_1x03_P2.54mm_Horizontal -> Connector_PinSocket_2.54mm:PinSocket_1x03_P2.54mm_Horizontal
- moved J5 9.83 mm to (112.5, 114.4), turned to 0 degrees
- moved J2 2.95 mm to (126.1, 136.3)
- moved G*** 0.85 mm to (112.5, 132.5)
Connections:
- D4 pad 2: /LIGHT-IO4-26 -> /PHOTO-IO2-24
- U5 pad 10: /Haptics-IN4 -> /Haptics-IN1
- U5 pad 11: /Haptics-ENA_PWM -> /Haptics-IN2
- U5 pad 12: /Haptics-ENB_PWM -> /Haptics-IN3
- U5 pad 13: /SDA -> /Haptics-ENA_PWM
- U5 pad 14: /SCL -> /Haptics-ENB_PWM
- U5 pad 16: /P0W-IO13-16 -> /Haptics-IN4
- U5 pad 23: /TRIG_2 -> /TRIG_4
- U5 pad 24: /LIGHT-IO4-26 -> /TRIG_3
- U5 pad 25: /IO0 -> /PHOTO-IO2-24
- U5 pad 26: /PHOTO-IO2-24 -> /LIGHT-IO4-26
- U5 pad 33: /TRIG_3 -> /SDA
- U5 pad 36: /ECHO_4 -> /SCL
- U5 pad 37: /TRIG_4 -> /ECHO_4
- U5 pad 4: /ECHO_1 -> /IO0
- U5 pad 5: /ECHO_2 -> /P0W-IO13-16
- U5 pad 7: /Haptics-IN1 -> /ECHO_2
- U5 pad 8: /Haptics-IN2 -> /ECHO_1
- U5 pad 9: /Haptics-IN3 -> /TRIG_2
Routing:
- net /TRIG_2: track 71.3 -> 48.9 mm, vias 2 -> 0
- net /SDA: track 100.0 -> 121.5 mm
- net +5V: track 270.5 -> 254.3 mm
- net /P0W-IO13-16: track 82.4 -> 94.4 mm, vias 0 -> 2
- net /TRIG_4: track 42.2 -> 32.3 mm, vias 0 -> 1
- net /PHOTO-IO2-24: track 110.7 -> 101.2 mm, vias 2 -> 0
- net /IO0: track 152.4 -> 159.7 mm
- net /ECHO_2: track 58.8 -> 53.0 mm
- net /LIGHT-IO4-26: track 105.8 -> 100.7 mm, vias 4 -> 0
- net /SCL: track 125.9 -> 121.2 mm, vias 4 -> 1
- net /TRIG_3: track 54.8 -> 50.1 mm, vias 0 -> 2
- net /EN: track 127.9 -> 123.8 mm
- net /TRIG_1: track 52.7 -> 48.8 mm
- net /Haptics-IN2: track 102.4 -> 98.4 mm
- net /Haptics-IN3: track 98.8 -> 94.9 mm
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
Commit message: re-routing rev 2.0
Parts:
- removed D4: LED, LED_SMD:LED_0805_2012Metric
- removed J4: Conn_01x08_Socket, Connector_PinSocket_2.54mm:PinSocket_1x08_P2.54mm_Vertical
- removed J6: Conn_01x02_Pin, Connector_PinSocket_2.54mm:PinSocket_1x02_P2.54mm_Vertical
- removed L1: Conn_01x06_Socket, Connector_PinSocket_2.54mm:PinSocket_1x06_P2.54mm_Horizontal
- removed R12: 1k, Resistor_SMD:R_0805_2012Metric
- added H1: MountingHole, MountingHole:MountingHole_2.2mm_M2, F.Cu at (117.8, 51.8)
- added H2: MountingHole, MountingHole:MountingHole_2.2mm_M2, F.Cu at (196.2, 51.8)
- added H3: MountingHole, MountingHole:MountingHole_2.2mm_M2, F.Cu at (117.8, 135.8)
- added H4: MountingHole, MountingHole:MountingHole_2.2mm_M2, F.Cu at (196.2, 135.8)
- J3: value Conn_01x02_Pin -> Screw_Terminal_01x03; footprint Connector_PinSocket_2.54mm:PinSocket_1x02_P2.54mm_Vertical -> TerminalBlock_Phoenix:TerminalBlock_Phoenix_PT-1,5-3-3.5-H_1x03_P3.50mm_Horizontal
- J5: value Conn_01x03_Socket -> Conn_01x04_Socket; footprint Connector_PinSocket_2.54mm:PinSocket_1x03_P2.54mm_Horizontal -> Connector_PinSocket_2.54mm:PinSocket_1x04_P2.54mm_Vertical
- moved D6 78.7 mm to (191.9, 107.4)
- moved R13 78.7 mm to (194.2, 111.6)
- moved J5 50.7 mm to (137.2, 70.1), turned to 180 degrees
- moved C1 44.1 mm to (177.8, 98.2), turned to 90 degrees
- moved Boot1 41.5 mm to (193.8, 99.4)
- moved Reset1 40.6 mm to (193.8, 89.2)
- moved C2 29.8 mm to (177.5, 91.0)
- moved S3 25.8 mm to (190.2, 80.0)
- moved J1 25.8 mm to (195.8, 122.0), turned to 90 degrees
- moved R5 25.1 mm to (180.0, 63.2)
- moved D2 24.5 mm to (190.8, 125.8)
- moved R6 24.2 mm to (180.8, 65.5), turned to 0 degrees
- moved R1 23.3 mm to (128.5, 57.2)
- moved R2 23.0 mm to (133.2, 59.5)
- moved S4 21.4 mm to (190.2, 65.8)
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Connections:
- Boot1 pad 2: /EN -> /BOOT
- C1 pad 1: /IO0 -> /EN
- C2 pad 1: /EN -> /BOOT
- C4 pad 1: /IO0 -> /BOOT
- J2 pad 1: /Haptics-IN1 -> /Haptics-ENA_PWM
- J2 pad 2: /Haptics-IN2 -> /Haptics-ENB_PWM
- J2 pad 3: /Haptics-IN3 -> /Haptics-IN1
- J2 pad 4: /Haptics-IN4 -> /Haptics-IN2
- J2 pad 5: /Haptics-ENA_PWM -> /Haptics-IN3
- J2 pad 6: /Haptics-ENB_PWM -> /Haptics-IN4
- J3 pad 1: /SDA -> +3.3V
- J3 pad 2: /SCL -> +5V
- J5 pad 2: +5V -> GND
- J5 pad 3: GND -> /SCL
- Q2 pad 3: /IO0 -> /BOOT
- R20 pad 2: /IO0 -> /BOOT
- Reset1 pad 2: /IO0 -> /EN
- U5 pad 10: /Haptics-IN1 -> /TRIG_1
- U5 pad 11: /Haptics-IN2 -> /TRIG_2
- U5 pad 12: /Haptics-IN3 -> /Haptics-ENA_PWM
- U5 pad 13: /Haptics-ENA_PWM -> /Haptics-ENB_PWM
- U5 pad 14: /Haptics-ENB_PWM -> /Haptics-IN1
- U5 pad 16: /Haptics-IN4 -> /Haptics-IN2
- U5 pad 23: /TRIG_4 -> /Haptics-IN3
- U5 pad 24: /TRIG_3 -> /Haptics-IN4
- U5 pad 25: /PHOTO-IO2-24 -> /BOOT
- U5 pad 31: /ECHO_3 -> /TRIG_3
- U5 pad 33: /SDA -> /ECHO_3
- U5 pad 36: /SCL -> /TRIG_4
- U5 pad 4: /IO0 -> /PHOTO-IO2-24
- U5 pad 6: /TRIG_1 -> /ECHO_1
- U5 pad 8: /ECHO_1 -> /SDA
- U5 pad 9: /TRIG_2 -> /SCL
Routing:
- net /IO0: track 159.7 -> 0.00 mm, vias 4 -> 0
- net /SCL: track 121.2 -> 18.6 mm, vias 1 -> 0
- net /SDA: track 121.5 -> 19.1 mm, vias 1 -> 0
- net /BOOT: track 0.00 -> 75.0 mm, vias 0 -> 2
- net /USB_DP: track 113.8 -> 80.2 mm
- net +5V: track 254.3 -> 221.5 mm, vias 3 -> 6
- net /Wheel_L_LPWM: track 102.9 -> 73.2 mm
- net /LIGHT-IO4-26: track 100.7 -> 71.1 mm
- net /Wheel_R_LPWM: track 106.7 -> 77.6 mm
- net /Wheel_L_RPWM: track 104.7 -> 75.7 mm
- net /Wheel_R_RPWM: track 108.1 -> 79.4 mm
- net /TRIG_3: track 50.1 -> 22.6 mm, vias 2 -> 0
- net /ECHO_3: track 32.9 -> 9.20 mm
- net /Haptics-IN1: track 103.2 -> 80.1 mm
- net /ECHO_1: track 50.5 -> 28.0 mm, vias 0 -> 2
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Other:
- board size 98 x 98 mm -> 84.9 x 90.5 mm
- board text added: "3.3V 5V GND"
- board text added: "HAPENA HAPENB HAPIN1 HAPIN2 HAPIN3 HAPIN4 POW PHOTO LIGHT WHEELLL WHEELLR WHEELRL WHEELRR"

Commit message: rev 2.0 PCB official
Parts:
- added D4: LED_YELLOW, LED_SMD:LED_0805_2012Metric, F.Cu at (153.8, 84.8)
- added D7: LED_BLUE, LED_SMD:LED_0805_2012Metric, F.Cu at (147.5, 73.9)
- added J4: Conn_01x02_Pin, Connector_PinSocket_2.54mm:PinSocket_1x02_P2.54mm_Horizontal, F.Cu at (124.7, 89.0)
- added R12: 10k, Resistor_SMD:R_0805_2012Metric, F.Cu at (149.0, 84.7)
- added R15: 10k, Resistor_SMD:R_0805_2012Metric, F.Cu at (144.5, 73.8)
- J2: value Conn_01x15_Socket -> Conn_01x16_Socket; footprint Connector_PinSocket_2.54mm:PinSocket_1x15_P2.54mm_Horizontal -> Connector_PinSocket_2.54mm:PinSocket_1x16_P2.54mm_Horizontal
- J3: value Screw_Terminal_01x03 -> Conn_01x03_Pin; footprint TerminalBlock_Phoenix:TerminalBlock_Phoenix_PT-1,5-3-3.5-H_1x03_P3.50mm_Horizontal -> Connector_JST:JST_XH_S3B-XH-A_1x03_P2.50mm_Horizontal
- moved J3 12.8 mm to (123.7, 99.8)
- moved G*** 11.6 mm to (121.6, 116.4)
Connections:
- J2 pad 1: /Haptics-ENA_PWM -> /Haptics-IN1
- J2 pad 2: /Haptics-ENB_PWM -> /Haptics-IN2
- J2 pad 3: /Haptics-IN1 -> /Haptics-IN3
- J2 pad 4: /Haptics-IN2 -> /Haptics-IN4
- J2 pad 5: /Haptics-IN3 -> unconnected-(J2-Pin_5-Pad5)
- J2 pad 6: /Haptics-IN4 -> unconnected-(J2-Pin_6-Pad6)
- J3 pad 1: +3.3V -> GND
- J3 pad 2: +5V -> +3.3V
- J3 pad 3: GND -> +5V
- U5 pad 12: /Haptics-ENA_PWM -> /LED_BLUE
- U5 pad 13: /Haptics-ENB_PWM -> /LED_YELLOW
Routing:
- net /Haptics-ENA_PWM: track 84.6 -> 0.00 mm
- net /Haptics-ENB_PWM: track 82.6 -> 0.00 mm
- net /LED_YELLOW: track 0.00 -> 48.7 mm, vias 0 -> 1
- net /LED_BLUE: track 0.00 -> 44.1 mm, vias 0 -> 1
- net +5V: track 221.5 -> 243.9 mm
- net GND: track 123.4 -> 130.5 mm, vias 19 -> 21
- net Net-(D4-K): track 0.00 -> 5.53 mm
- net /Haptics-IN4: track 88.7 -> 93.7 mm
- net /USB_DN: track 73.2 -> 78.1 mm
- net /P0W-IO13-16: track 110.9 -> 107.1 mm
- net /Haptics-IN3: track 89.1 -> 92.7 mm
- net /PHOTO-IO2-24: track 118.3 -> 114.8 mm
- net Net-(D7-K): track 0.00 -> 2.98 mm
- net /Haptics-IN2: track 81.9 -> 84.7 mm
- net /Wheel_R_RPWM: track 79.4 -> 76.8 mm
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Other:
- board text added: "5V TRIG ECHO GND"
- board text added: "FORWARD Group 25 Main PCB Rev 2.0"
- board text added: "GND 3.3V 5V"
- board text added: "HAPIN1 HAPIN2 HAPIN3 HAPIN4 X X POW PHOTO LIGHT WHEELLL WHEELLR WHEELRL WHEELRR GND 3.3V X"
- board text added: "I2S"
- board text added: "IMU"
- board text added: "SDA SCL GND 3.3V"
- board text removed: "3.3V 5V GND"
- board text removed: "HAPENA HAPENB HAPIN1 HAPIN2 HAPIN3 HAPIN4 POW PHOTO LIGHT WHEELLL WHEELLR WHEELRL WHEELRR"
