File: FORWARD-MAIN/FORWARD-PCB.kicad_sch (KiCad schematic)
At the start: 43 parts, among them J1 USB_B_Micro, J2 Conn_01x03_Socket, J3 Conn_01x13_Socket, J4 Conn_01x08_Socket, Q1 SS8050-G, Q2 SS8050-G, U2 CP2102N-Axx-xQFN28, U5 ESP32-WROOM-32D

Commit message: a good iteration!
Parts:
- added R3: 1k, Resistor_SMD:R_0805_2012Metric, symbol Device:R_US
- added R4: 2k, Resistor_SMD:R_0805_2012Metric, symbol Device:R_US
- added S2: Conn_01x04_Socket, Connector_JST:JST_EH_S4B-EH_1x04_P2.50mm_Horizontal, symbol Connector:Conn_01x04_Socket
Connections:
- net +5V: now also S2.1 (Pin_1)
- net ECHO_1: now also U5.4 (SENSOR_VP); no longer U5.23 (IO15)
- net GND: now also R4.2, S2.4 (Pin_4)
- net LIGHT-IO4-26: now also U5.26 (IO4); no longer U5.29 (IO5)
- net ECHO_2: now reaches U5.5 (SENSOR_VN)
- net ECHO_2: now also R3.2, R4.1
- net Haptics-IO25 renamed Haptics-IN1
- net Haptics-IO26 renamed Haptics-IN2
- net Haptics-IO27 renamed Haptics-IN3
- net Haptics-IO32 renamed Haptics-IN4
- net Haptics-IO33 renamed Haptics-ENA_PWM
- net Haptics-IO35 renamed Haptics-ENB_PWM
- net Wheels-IO16-27 renamed Wheels_LPWM
- net Wheels_LPWM: now also U5.28 (IO17); no longer U5.26 (IO4)
- net Wheels-IO17-28 renamed IO16-27
- net IO16-27: now also U5.29 (IO5); no longer U5.27 (IO16)
- net Wheels-IO18-30 renamed IO18-30
- net Wheels-IO5-29 renamed Wheels-RPWM
- net Wheels-RPWM: now also U5.27 (IO16); no longer U5.28 (IO17)
- new net: R3.1, S2.3 (Pin_3)
- new net TRIG_2: S2.2 (Pin_2), U5.23 (IO15)
- no-connect marks 30 -> 28
Other:
- note added: "Direction Control"
- note added: "Speed Control"
- moved on the sheet: J4, R16, R17

Commit message: ready to order (i think)
Parts:
- removed J2: Conn_01x03_Socket, Connector_PinHeader_2.54mm:PinHeader_1x03_P2.54mm_Horizontal, symbol Connector:Conn_01x03_Socket
- added C4: 0.1uF, Capacitor_SMD:C_0805_2012Metric, symbol Device:C_Small
- added D4: LED, LED_SMD:LED_0805_2012Metric, symbol Device:LED
- added J5: Screw_Terminal_01x03, TerminalBlock_Phoenix:TerminalBlock_Phoenix_MPT-0,5-3-2.54_1x03_P2.54mm_Horizontal, symbol Connector:Screw_Terminal_01x03
- added R20: 10k, Resistor_SMD:R_0805_2012Metric, symbol Device:R_US
- L1: footprint Connector_JST:JST_PH_S6B-PH-K_1x06_P2.00mm_Horizontal -> Connector_JST:JST_EH_S6B-EH_1x06_P2.50mm_Horizontal
Connections:
- net +3.3V: now also J5.1 (Pin_1), R20.1; no longer C3.1, C5.1, R14.2, U2.6 (VDD), U2.7 (VREGIN)
- net +5V: now also C3.1, C5.1, R14.2, U2.6 (VDD), U2.7 (VREGIN), J5.2 (Pin_2)
- net GND: now also U5.15 (GND), C4.2, J5.3 (Pin_3)
- net IO0: now also C1.1, Reset1.2, C4.1, D4.2 (A), R20.2; no longer U5.25 (IO0)
- net IO16-27 renamed Wheel_R_LPWM
- net IO18-30 renamed Wheel_R_RPWM
- net RST: no longer names the net of R14.1, U2.9 (~{RST})
- net RST: no longer C1.1, Reset1.2
- net Wheels-RPWM renamed Wheel_L_LPWM
- net Wheels_LPWM renamed Wheel_L_RPWM
- new net: D4.1 (K), U5.25 (IO0)
- no-connect marks 28 -> 27
Other:
- note added: "output only"
- note removed: "i/p from PCB 2"
- moved on the sheet: C10, R18
