File: FORWARD-POWER/FORWARD-POWER.kicad_pcb (KiCad board)
At the start: 2 copper layers, 77 x 32 mm, 20 parts, among them J1 Conn_01x03_Pin, J2 Conn_01x03_Pin, J3 Conn_01x01_Pin, J4 Screw_Terminal_01x04, J5 Conn_01x01_Pin, U1 AMS1117-3.3, U2 AMS1117-5.0

Commit message: PCB order rev 1.0
Parts:
- removed D2, D3: D, Diode_THT:D_A-405_P7.62mm_Horizontal
- removed J5: Conn_01x01_Pin, Connector_PinHeader_2.54mm:PinHeader_1x01_P2.54mm_Vertical
- removed VR2: LM7805MPX_NOPB, footprints:VREG_LM7805MPX_NOPB
- added C5: 100uF, Capacitor_SMD:C_Elec_6.3x7.7, F.Cu at (202.8, 112.5)
- added D4: 1N5822, footprints:DIOAD1990W125L900D530, F.Cu at (217.1, 123.5)
- added G***: LOGO, footprints:lambda, F.Cu at (191.0, 123.0)
- added L2: SRR7045-331M, footprints:IND_BOURNS_SRR7045, F.Cu at (235.5, 122.5)
- added U3: LM2576-5.0WT, Package_TO_SOT_THT:TO-220-5_P3.4x3.7mm_StaggerEven_Lead3.8mm_Vertical, F.Cu at (213.8, 112.2)
- C4: value 220uF -> UWT1E331MNL1GS; footprint Capacitor_SMD:C_0805_2012Metric -> footprints:PCAP_8x10-ELECT_NCA
- moved C4 26.1 mm to (230.2, 112.5)
- moved H2 9.25 mm to (177.5, 126.0)
- moved H4 9.25 mm to (248.5, 126.0)
- moved C1 4.34 mm to (195.6, 100.5)
- moved C2 4.34 mm to (213.6, 97.5)
- moved C3 4.34 mm to (234.6, 91.5)
- moved D1 4.34 mm to (215.6, 90.5)
- moved J3 4.34 mm to (207.6, 96.5)
- moved R1 4.34 mm to (210.6, 91.5)
- moved U1 4.34 mm to (225.6, 93.5)
- moved U2 4.34 mm to (198.6, 93.5)
- moved H1 0.50 mm to (177.5, 90.8)
Connections:
- C4 pad 1: GND -> +5V
- C4 pad 2: Net-(D2-A) -> GND3
- J1 pad 1: GND -> GND3
- J4 pad 2: GND -> GND3
Routing:
- net GND: track 84.5 -> 30.0 mm, vias 13 -> 7
- net GND3: track 0.00 -> 47.1 mm, vias 0 -> 4
- net Net-(U3-OUTPUT): track 0.00 -> 31.9 mm
- net +5V: track 21.9 -> 51.4 mm
- net Net-(D2-A): track 27.4 -> 0.00 mm
- net +12V: track 59.4 -> 72.3 mm
- net +3.3V: track 23.6 -> 26.3 mm
- net +6V: track 15.3 -> 16.1 mm
- added copper zone on B.Cu, net GND3
Other:
- board size 77 x 32 mm -> 77 x 41.2 mm
