File: FORWARD-POWER/FORWARD-POWER.kicad_pcb (KiCad board)
At the start: 2 copper layers, 77 x 41.2 mm, 21 parts, among them J1 Conn_01x03_Pin, J2 Conn_01x03_Pin, J3 Conn_01x01_Pin, J4 Screw_Terminal_01x04, U1 AMS1117-3.3, U2 AMS1117-5.0, U3 LM2576-5.0WT

Commit message: rev 2.0 PCB official
Parts:
- removed J1: Conn_01x03_Pin, Connector_PinHeader_2.54mm:PinHeader_1x03_P2.54mm_Vertical
- added J5: Screw_Terminal_01x04, TerminalBlock_Phoenix:TerminalBlock_Phoenix_MKDS-3-4-5.08_1x04_P5.08mm_Horizontal, F.Cu at (185.1, 123.5)
- added J6: Conn_01x03_Pin, Connector_JST:JST_XH_S3B-XH-A-1_1x03_P2.50mm_Horizontal, F.Cu at (248.8, 116.0)
- J2: footprint Connector_PinHeader_2.54mm:PinHeader_1x03_P2.54mm_Vertical -> Connector_JST:JST_XH_S3B-XH-A-1_1x03_P2.50mm_Horizontal
- moved G*** 44.7 mm to (230.0, 101.2)
- moved J2 5.39 mm to (248.8, 101.5), turned to 90 degrees
- moved H3 5.25 mm to (253.8, 90.8)
- moved H4 5.25 mm to (253.8, 126.0)
- moved J4 3.03 mm to (183.5, 96.3)
Connections:
- J2 pad 2: /anet -> +3.3V
- J2 pad 3: +3.3V -> /anet
- J4 pad 2: GND3 -> +6V
- J4 pad 3: +6V -> GND3
Routing:
- net +12V: track 72.3 -> 102.5 mm
- net +3.3V: track 26.3 -> 39.1 mm
- net +5V: track 51.4 -> 58.0 mm
- net GND: track 30.0 -> 34.8 mm
- net /anet: track 60.0 -> 64.7 mm
- net GND3: track 47.1 -> 45.0 mm
- net +6V: track 16.1 -> 16.7 mm
Other:
- board size 77 x 41.2 mm -> 82.2 x 41.2 mm
- board text added: "5V 3.3V GND"
- board text added: "BTS7960"
- board text added: "Control PCB"
- board text added: "GND-6 6V GND-12 12V"
- board text added: "Main PCB"
- board text added: "Power Supply"
- board text removed: "3.3V 5V GND"
- board text removed: "GND-6 GND-12 6V 12V"
