File: FORWARD-POWER/FORWARD-POWER.kicad_sch (KiCad schematic)
At the start: 22 parts, among them J1 Conn_01x02_Pin, J2 Conn_01x03_Pin, U3 AMS1117-3.3, U4 TPS63070RNMR

Commit message: itried
Parts:
- removed C11, Cout1: 47uF, Capacitor_SMD:C_0805_2012Metric, symbol Device:C_Small
- removed C12, C4: 100nF, Capacitor_SMD:C_0805_2012Metric, symbol Device:C_Small
- removed Coutx1: 10uF, Capacitor_SMD:C_0805_2012Metric, symbol Device:C_Small
- removed D4: LED, LED_SMD:LED_0805_2012Metric, symbol Device:LED
- removed J1: Conn_01x02_Pin, Connector_JST:JST_PH_S2B-PH-K_1x02_P2.00mm_Horizontal, symbol Connector:Conn_01x02_Pin
- removed L2: 1.5uH, Inductor_SMD:L_0805_2012Metric, symbol Device:L
- removed Renable1: 10k, Resistor_SMD:R_0805_2012Metric, symbol Device:R_US
- removed Rfbb1, Rpgood1: 100k, Resistor_SMD:R_0805_2012Metric, symbol Device:R_US
- removed Rfbt1: 523k, Resistor_SMD:R_0805_2012Metric, symbol Device:R_US
- removed TP1: TestPoint, TestPoint:TestPoint_Pad_1.5x1.5mm, symbol Connector:TestPoint
- removed U4: TPS63070RNMR, pcb-footprints:VREG_TPS63070RNMR, symbol TPS63070RNMR:TPS63070RNMR
- removed VR1: LM3940IMP-3.3_NOPB, LM3940IMP-3.3_NOPB:VREG_LM3940IMP-3.3_NOPB, symbol LM3940IMP-3.3_NOPB:LM3940IMP-3.3_NOPB
- added C5: 220uF, Capacitor_SMD:C_0805_2012Metric, symbol Device:C_Small
- added J1: Conn_01x03_Pin, Connector_PinHeader_2.54mm:PinHeader_1x03_P2.54mm_Vertical, symbol Connector:Conn_01x03_Pin
- added J4: Screw_Terminal_01x04, TerminalBlock_Phoenix:TerminalBlock_Phoenix_MKDS-1,5-4-5.08_1x04_P5.08mm_Horizontal, symbol Connector:Screw_Terminal_01x04
- added R2: 1k, Resistor_SMD:R_0805_2012Metric, symbol Device:R_US
- added R3: 5k, Resistor_SMD:R_0805_2012Metric, symbol Device:R_US
- added VR2: LM7805MPX_NOPB, footprints:VREG_LM7805MPX_NOPB, symbol LM7805MPX_NOPB:LM7805MPX_NOPB
- J2: footprint Connector_JST:JST_PH_S3B-PH-K_1x03_P2.00mm_Horizontal -> Connector_PinHeader_2.54mm:PinHeader_1x03_P2.54mm_Vertical
Connections:
- net +5V: now also C5.2, J1.2 (Pin_2); no longer C6.1, J2.2 (Pin_2), R15.1, TP2.1, U3.3 (VI)
- net +6V: now also J4.3 (Pin_3), R2.1
- net GND: now also J1.1 (Pin_1), J4.1 (Pin_1), J4.2 (Pin_2), R3.1, VR2.2 (GND_2), VR2.4 (GND_4)
- new net: C5.1, VR2.3 (OUTPUT)
- new net +12V: J1.3 (Pin_3), J4.4 (Pin_4), VR2.1 (INPUT)
- new net anet: C6.1, J2.2 (Pin_2), R15.1, R2.2, R3.2, TP2.1, U3.3 (VI)
Other:
- note added: "to Control PCB"
- note added: "to main PCB"
- note removed: "Power Supply & Voltage Regulators"
- note removed: "bypass"
- moved on the sheet: C6, C7, D4, J2, R15, TP2, U3

Commit message: regulator pcb done
Parts:
- removed R2: 1k, Resistor_SMD:R_0805_2012Metric, symbol Device:R_US
- removed R3: 5k, Resistor_SMD:R_0805_2012Metric, symbol Device:R_US
- added C1: 47uF, Capacitor_SMD:C_0805_2012Metric, symbol Device:C_Small
- added H1, H2, H3, H4: MountingHole, MountingHole:MountingHole_2.2mm_M2, symbol Mechanical:MountingHole
- added U2: AMS1117-5.0, Package_TO_SOT_SMD:SOT-223-3_TabPin2, symbol Regulator_Linear:AMS1117-5.0
Connections:
- net +6V: now also C1.1, U2.3 (VI)
- net GND: now also C1.2, U2.1 (GND)
- net anet: now also U2.2 (VO)

Commit message: ready to order (i think)
Parts:
- removed C5: 220uF, Capacitor_SMD:C_0805_2012Metric, symbol Device:C_Small
- added C4: 220uF, Capacitor_SMD:C_0805_2012Metric, symbol Device:C_Small
- added D2: D, Diode_SMD:D_0805_2012Metric, symbol Device:D
Connections:
- net +5V: now also D2.1 (K)
- net GND: now also C4.1
- net at VR2.3 (OUTPUT): now also C4.2, D2.2 (A)
Changed lines of the file:
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@@
+	)
+	(junction
+		(at 163.83 142.24)
+		(diameter 0)
+		(color 0 0 0 0)
 	)
 	(junction
@@
 	)
 	(junction
-		(at 173.99 142.24)
+		(at 184.15 142.24)
 		(diameter 0)
 		(color 0 0 0 0)
@@
 	(wire
 		(pts
-			(xy 173.99 142.24) (xy 168.91 142.24)
-		)
-		(stroke
-			(width 0)
-			(type default)
-		)
-	)
-	(wire
-		(pts
 			(xy 90.17 124.46) (xy 90.17 127)
 		)
@@
 	(wire
 		(pts
+			(xy 177.8 142.24) (xy 184.15 142.24)
+		)
+		(stroke
+			(width 0)
+			(type default)
+		)
+	)
+	(wire
+		(pts
 			(xy 123.19 72.39) (xy 132.08 72.39)
 		)
@@
 	(wire
 		(pts
+			(xy 163.83 142.24) (xy 163.83 144.78)
+		)
+		(stroke
+			(width 0)
+			(type default)
+		)
+	)
+	(wire
+		(pts
 			(xy 132.08 72.39) (xy 132.08 81.28)
 		)
@@
 	(wire
 		(pts
+			(xy 163.83 153.67) (xy 163.83 149.86)
+		)
+		(stroke
+			(width 0)
+			(type default)
+		)
+	)
+	(wire
+		(pts
 			(xy 156.21 149.86) (xy 156.21 147.32)
 		)
@@
 		(pts
 			(xy 156.21 153.67) (xy 156.21 149.86)
+		)
+		(stroke
+			(width 0)
+			(type default)
+		)
+	)
+	(wire
+		(pts
+			(xy 163.83 142.24) (xy 170.18 142.24)
 		)
 		(stroke
@@
 	)
 	(symbol
+		(lib_id "Device:D")
+		(at 173.99 142.24 180)
+		(unit 1)
+		(exclude_from_sim no)
+		(in_bom yes)
+		(on_board yes)
+		(dnp no)
+		(fields_autoplaced yes)
+		(property "Reference" "D2"
+			(at 173.99 135.89 0)
+			(effects
+				(font
+					(size 1.27 1.27)
+				)
+			)
+		)
+		(property "Value" "D"
+			(at 173.99 138.43 0)
+			(effects
+				(font
+					(size 1.27 1.27)
+				)
+			)
+		)
+		(property "Footprint" "Diode_SMD:D_0805_2012Metric"
+			(at 173.99 142.24 0)
+			(effects
+				(font
+					(size 1.27 1.27)
+				)
+				(hide yes)
+			)
+		)
+		(property "Datasheet" "~"
+			(at 173.99 142.24 0)
+			(effects
+				(font
+					(size 1.27 1.27)
+				)
+				(hide yes)
+			)
+		)
+		(property "Description" "Diode"
+			(at 173.99 142.24 0)
+			(effects
+				(font
+					(size 1.27 1.27)
+				)
+				(hide yes)
+			)
+		)
+		(property "Sim.Device" "D"
+			(at 173.99 142.24 0)
+			(effects
+				(font
+					(size 1.27 1.27)
+				)
+				(hide yes)
+			)
+		)
+		(property "Sim.Pins" "1=K 2=A"
+			(at 173.99 142.24 0)
+			(effects
+				(font
+					(size 1.27 1.27)
+				)
+				(hide yes)
+			)
+		)
+		(pin "1"
+		)
+		(pin "2"
+		)
+		(instances
+			(project ""
+				(path "/ce51f21b-ae90-4513-bbba-00af99e3d46b"
+					(reference "D2")
+					(unit 1)
+				)
+			)
+		)
+	)
+	(symbol
 		(lib_id "power:+6V")
 		(at 85.09 123.19 0)
@@
 	(symbol
 		(lib_id "power:PWR_FLAG")
-		(at 173.99 142.24 270)
+		(at 184.15 142.24 270)
 		(unit 1)
 		(exclude_from_sim no)
@@
 		(fields_autoplaced yes)
 		(property "Reference" "#FLG03"
-			(at 175.895 142.24 0)
+			(at 186.055 142.24 0)
 			(effects
 				(font
@@
 		)
 		(property "Value" "PWR_FLAG"
-			(at 177.8 142.2399 90)
+			(at 187.96 142.2399 90)
 			(effects
 				(font
@@
 		)
 		(property "Footprint" ""
-			(at 173.99 142.24 0)
+			(at 184.15 142.24 0)
 			(effects
 				(font
@@
 		)
 		(property "Datasheet" "~"
-			(at 173.99 142.24 0)
+			(at 184.15 142.24 0)
 			(effects
 				(font
@@
 		)
 		(property "Description" "Special symbol for telling ERC where power comes from"
-			(at 173.99 142.24 0)
+			(at 184.15 142.24 0)
 			(effects
 				(font
@@
 	)
 	(symbol
-		(lib_id "Device:C_Small")
-		(at 166.37 142.24 90)
-		(unit 1)
-		(exclude_from_sim no)
-		(in_bom yes)
-		(on_board yes)
-		(dnp no)
-		(fields_autoplaced yes)
-		(property "Reference" "C5"
-			(at 166.3763 135.89 90)
-			(effects
-				(font
-					(size 1.27 1.27)
-				)
-			)
-		)
-		(property "Value" "220uF"
-			(at 166.3763 138.43 90)
-			(effects
-				(font
-					(size 1.27 1.27)
-				)
-			)
-		)
-		(property "Footprint" "Capacitor_SMD:C_0805_2012Metric"
-			(at 166.37 142.24 0)
-			(effects
-				(font
-					(size 1.27 1.27)
-				)
-				(hide yes)
-			)
-		)
-		(property "Datasheet" "~"
-			(at 166.37 142.24 0)
-			(effects
-				(font
-					(size 1.27 1.27)
-				)
-				(hide yes)
-			)
-		)
-		(property "Description" "Unpolarized capacitor, small symbol"
-			(at 166.37 142.24 0)
-			(effects
-				(font
-					(size 1.27 1.27)
-				)
-				(hide yes)
-			)
-		)
-		(pin "2"
-		)
-		(pin "1"
-		)
-		(instances
-			(project ""
-				(path "/ce51f21b-ae90-4513-bbba-00af99e3d46b"
-					(reference "C5")
-					(unit 1)
-				)
-			)
-		)
-	)
-	(symbol
 		(lib_id "power:+3.3V")
 		(at 196.85 111.76 90)
@@
 	)
 	(symbol
+		(lib_id "power:GND")
+		(at 163.83 153.67 0)
+		(unit 1)
+		(exclude_from_sim no)
+		(in_bom yes)
+		(on_board yes)
+		(dnp no)
+		(fields_autoplaced yes)
+		(property "Reference" "#PWR06"
+			(at 163.83 160.02 0)
+			(effects
+				(font
+					(size 1.27 1.27)
+				)
+				(hide yes)
+			)
+		)
+		(property "Value" "GND"
+			(at 163.83 158.75 0)
+			(effects
+				(font
+					(size 1.27 1.27)
+				)
+			)
+		)
+		(property "Footprint" ""
+			(at 163.83 153.67 0)
+			(effects
+				(font
+					(size 1.27 1.27)
+				)
+				(hide yes)
+			)
+		)
+		(property "Datasheet" ""
+			(at 163.83 153.67 0)
+			(effects
+				(font
+					(size 1.27 1.27)
+				)
+				(hide yes)
+			)
+		)
+		(property "Description" ""
+			(at 163.83 153.67 0)
+			(effects
+				(font
+					(size 1.27 1.27)
+				)
+				(hide yes)
+			)
+		)
+		(pin "1"
+		)
+		(instances
+			(project "FORWARD-POWER"
+				(path "/ce51f21b-ae90-4513-bbba-00af99e3d46b"
+					(reference "#PWR06")
+					(unit 1)
+				)
+			)
+		)
+	)
+	(symbol
 		(lib_id "power:PWR_FLAG")
 		(at 163.83 114.3 0)
@@
 	)
 	(symbol
+		(lib_id "Device:C_Small")
+		(at 163.83 147.32 0)
+		(mirror x)
+		(unit 1)
+		(exclude_from_sim no)
+		(in_bom yes)
+		(on_board yes)
+		(dnp no)
+		(property "Reference" "C4"
+			(at 170.18 147.3137 90)
+			(effects
+				(font
+					(size 1.27 1.27)
+				)
+			)
+		)
+		(property "Value" "220uF"
+			(at 167.64 147.3137 90)
+			(effects
+				(font
+					(size 1.27 1.27)
+				)
+			)
+		)
+		(property "Footprint" "Capacitor_SMD:C_0805_2012Metric"
+			(at 163.83 147.32 0)
+			(effects
+				(font
+					(size 1.27 1.27)
+				)
+				(hide yes)
+			)
+		)
+		(property "Datasheet" "~"
+			(at 163.83 147.32 0)
+			(effects
+				(font
+					(size 1.27 1.27)
+				)
+				(hide yes)
+			)
+		)
+		(property "Description" "Unpolarized capacitor, small symbol"
+			(at 163.83 147.32 0)
+			(effects
+				(font
+					(size 1.27 1.27)
+				)
+				(hide yes)
+			)
+		)
+		(pin "2"
+		)
+		(pin "1"
+		)
+		(instances
+			(project "FORWARD-POWER"
+				(path "/ce51f21b-ae90-4513-bbba-00af99e3d46b"
+					(reference "C4")
+					(unit 1)
+				)
+			)
+		)
+	)
+	(symbol
 		(lib_id "Mechanical:MountingHole")
 		(at 190.5 81.28 0)
@@
 	(symbol
 		(lib_id "power:+5V")
-		(at 173.99 142.24 0)
+		(at 184.15 142.24 0)
 		(unit 1)
 		(exclude_from_sim no)
@@
 		(fields_autoplaced yes)
 		(property "Reference" "#PWR012"
-			(at 173.99 146.05 0)
+			(at 184.15 146.05 0)
 			(effects
 				(font
@@
 		)
 		(property "Value" "+5V"
-			(at 173.99 137.16 0)
+			(at 184.15 137.16 0)
 			(effects
 				(font
@@
 		)
 		(property "Footprint" ""
-			(at 173.99 142.24 0)
+			(at 184.15 142.24 0)
 			(effects
 				(font
@@
 		)
 		(property "Datasheet" ""
-			(at 173.99 142.24 0)
+			(at 184.15 142.24 0)
 			(effects
 				(font
@@
 		)
 		(property "Description" ""
-			(at 173.99 142.24 0)
-			(effects
-				(font
+			(at 184.15 142.24 0)
+			(effects
+				(font
