File: FORWARD-POWER/FORWARD-POWER.kicad_sch (KiCad schematic)
At the start: 20 parts, among them J1 Conn_01x03_Pin, J2 Conn_01x03_Pin, J3 Conn_01x01_Pin, J4 Screw_Terminal_01x04, J5 Conn_01x01_Pin, U2 AMS1117-5.0, U3 AMS1117-3.3

Commit message: PCB order rev 1.0
Parts:
- removed C4: 220uF, Capacitor_SMD:C_0805_2012Metric, symbol Device:C_Small
- removed D2, D3: D, Diode_THT:D_A-405_P7.62mm_Horizontal, symbol Device:D
- removed J5: Conn_01x01_Pin, Connector_PinHeader_2.54mm:PinHeader_1x01_P2.54mm_Vertical, symbol Connector:Conn_01x01_Pin
- removed VR2: LM7805MPX_NOPB, footprints:VREG_LM7805MPX_NOPB, symbol LM7805MPX_NOPB:LM7805MPX_NOPB
- added C4: UWT1E331MNL1GS, footprints:PCAP_8x10-ELECT_NCA, symbol PCAP330:UWT1E331MNL1GS
- added C5: 100uF, Capacitor_SMD:C_Elec_6.3x7.7, symbol Device:C_Small
- added D4: 1N5822, footprints:DIOAD1990W125L900D530, symbol 1N5822:1N5822
- added L2: SRR7045-331M, footprints:IND_BOURNS_SRR7045, symbol L330:SRR7045-331M
- added U3: LM2576-5.0WT, Package_TO_SOT_THT:TO-220-5_P3.4x3.7mm_StaggerEven_Lead3.8mm_Vertical, symbol LM2576-5.0WT:LM2576-5.0WT
Connections:
- net +12V: now also C5.1, U3.1 (VIN)
- net +5V: now also C4.1, L2.2, U3.4 (FEEDBACK)
- net GND: no longer J1.1 (Pin_1), J4.2 (Pin_2)
- new net: D4.C, L2.1, U3.2 (OUTPUT)
- new net GND3: C4.2, C5.2, D4.A, J1.1 (Pin_1), J4.2 (Pin_2), U3.3 (GROUND), U3.5 (*ON/OFF)
Other:
- moved on the sheet: C1, C6, C7, D4, H1, H2, H3, H4, J1, J2, J3, J4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

Commit message: rev 2.0 PCB official
Parts:
- removed J1: Conn_01x03_Pin, Connector_PinHeader_2.54mm:PinHeader_1x03_P2.54mm_Vertical, symbol Connector:Conn_01x03_Pin
- added J5: Screw_Terminal_01x04, TerminalBlock_Phoenix:TerminalBlock_Phoenix_MKDS-3-4-5.08_1x04_P5.08mm_Horizontal, symbol Connector:Screw_Terminal_01x04
- added J6: Conn_01x03_Pin, Connector_JST:JST_XH_S3B-XH-A-1_1x03_P2.50mm_Horizontal, symbol Connector:Conn_01x03_Pin
- J2: footprint Connector_PinHeader_2.54mm:PinHeader_1x03_P2.54mm_Vertical -> Connector_JST:JST_XH_S3B-XH-A-1_1x03_P2.50mm_Horizontal
Connections:
- net +12V: now also J5.1 (Pin_1), J5.2 (Pin_2), J6.3 (Pin_3)
- net +3.3V: now also J2.2 (Pin_2); no longer J2.3 (Pin_3)
- net +5V: now also J6.2 (Pin_2)
- net +6V: now also J4.2 (Pin_2); no longer J4.3 (Pin_3)
- net GND3: now also J4.3 (Pin_3), J5.3 (Pin_3), J5.4 (Pin_4), J6.1 (Pin_1); no longer J4.2 (Pin_2)
- net anet: now also J2.3 (Pin_3); no longer J2.2 (Pin_2)
Other:
- note added: "to Motor Drivers"
- moved on the sheet: J2
