File: FORWARD-CONTROLLER/MotorDriverPCB.kicadBefore_March_14_sch.kicad_sch (KiCad schematic)
At the start: 22 parts, among them J1 Conn_01x16_Pin, J2 Conn_02x04_Counter_Clockwise, J3 Conn_02x04_Counter_Clockwise, J4 Conn_01x03_Socket, J5 Conn_01x02_Socket, Q1 2N2219, U3 L298N

Commit message: the real motor rev 2.0
Parts:
- removed J1: Conn_01x16_Pin, Connector_PinHeader_2.54mm:PinHeader_1x16_P2.54mm_Horizontal, symbol Connector:Conn_01x16_Pin
- added J1: Conn_01x15_Pin, Connector_PinHeader_2.54mm:PinHeader_1x15_P2.54mm_Horizontal, symbol Connector:Conn_01x15_Pin
- added SW1: SW_DIP_x02, Button_Switch_SMD:SW_DIP_SPSTx02_Slide_KingTek_DSHP02TS_W7.62mm_P1.27mm, symbol Switch:SW_DIP_x02
- H1, H2: footprint Connector_JST:JST_XH_S2B-XH-A-1_1x02_P2.50mm_Horizontal -> TerminalBlock_Phoenix:TerminalBlock_Phoenix_MKDS-1,5-2-5.08_1x02_P5.08mm_Horizontal
Connections:
- net +12V: now also J4.2 (Pin_2), U3.9 (VSS); no longer J4.1 (Pin_1)
- net +3.3V: now also J1.15 (Pin_15)
- net +5V: now also J2.3 (Pin_3), J2.8 (Pin_8), J3.3 (Pin_3), J3.8 (Pin_8), J4.1 (Pin_1); no longer J2.5 (Pin_5), J2.7 (Pin_7), J3.5 (Pin_5), J3.7 (Pin_7), J4.2 (Pin_2), U3.11 (ENB), U3.6 (ENA), U3.9 (VSS)
- net GND: now also J2.1 (Pin_1), J3.1 (Pin_1), J1.14 (Pin_14); no longer J2.8 (Pin_8), J3.8 (Pin_8)
- net IN1U2: now also J3.4 (Pin_4), J1.10 (Pin_10); no longer J3.2 (Pin_2)
- net IN1U3: now also J1.2 (Pin_2)
- net IN2U2: now also J3.5 (Pin_5), J1.11 (Pin_11); no longer J3.1 (Pin_1)
- net IN2U3: now also J1.1 (Pin_1)
- net IN3U2: now also J2.4 (Pin_4), J1.12 (Pin_12); no longer J2.2 (Pin_2)
- net IN3U3: now also J1.4 (Pin_4)
- net IN4U2: now also J2.5 (Pin_5), J1.13 (Pin_13); no longer J2.1 (Pin_1)
- net IN4U3: now also J1.3 (Pin_3)
- net LIGHT: now also J1.9 (Pin_9)
- net PHOTO: now also J1.8 (Pin_8)
- net POW: now also J1.7 (Pin_7)
- new net ENAU3: SW1.1, U3.6 (ENA)
- new net ENBU3: SW1.2, U3.11 (ENB)
- new net SW1U3: J1.5 (Pin_5), SW1.4
- new net SW2U3: J1.6 (Pin_6), SW1.3
- no-connect marks 7 -> 4
Other:
- note added: "Switches between Drivers and MCU"
