File: FORWARD-CONTROLLER/MotorDriverPCB.kicad_pcb (KiCad board)
At the start: 4 copper layers, 70.2 x 54.2 mm, 22 parts, among them J1 Conn_01x14_Pin, J2 Conn_02x04_Counter_Clockwise, J3 Conn_02x04_Counter_Clockwise, J4 Conn_01x03_Socket, Q1 2N2219, SW1 SW_DIP_x02, U3 L298N

Commit message: the real motor rev 2.0
Parts:
- removed C4: 220uF, Capacitor_SMD:C_0805_2012Metric
- removed D10, D15, D16, D17, D18, D9: 1N4002, Diode_SMD:D_0805_2012Metric
- removed SW1: SW_DIP_x02, Button_Switch_SMD:SW_DIP_SPSTx02_Slide_KingTek_DSHP02TS_W7.62mm_P1.27mm
- added D1: STTH212U, Diode_SMD:D_SMB, F.Cu at (114.6, 80.5)
- added D2: STTH212U, Diode_SMD:D_SMB, F.Cu at (122.5, 76.2)
- added D3: STTH212U, Diode_SMD:D_SMB, F.Cu at (115.0, 88.0)
- added D4: STTH212U, Diode_SMD:D_SMB, F.Cu at (115.0, 94.8)
- added D5: STTH212U, Diode_SMD:D_SMB, F.Cu at (126.1, 95.0)
- added D6: STTH212U, Diode_SMD:D_SMB, F.Cu at (124.2, 88.0)
- added G***: LOGO, Lambda:lambda, F.Cu at (153.2, 79.0)
- added J5: Conn_01x02_Socket, Connector_PinSocket_2.54mm:PinSocket_1x02_P2.54mm_Horizontal, F.Cu at (112.0, 105.5)
- added R3: 10k, Resistor_SMD:R_0805_2012Metric, F.Cu at (133.8, 69.4)
- added REF**: MountingHole_2.1mm, MountingHole:MountingHole_2.1mm, F.Cu at (170.0, 60.0)
- added REF**: MountingHole_2.1mm, MountingHole:MountingHole_2.1mm, F.Cu at (100.0, 107.0)
- added REF**: MountingHole_2.1mm, MountingHole:MountingHole_2.1mm, F.Cu at (100.0, 60.0)
- added REF**: MountingHole_2.1mm, MountingHole:MountingHole_2.1mm, F.Cu at (170.0, 107.0)
- D7, D8: value 1N4002 -> STTH212U; footprint Diode_SMD:D_0805_2012Metric -> Diode_SMD:D_SMB
- H1, H2: footprint TerminalBlock_Phoenix:TerminalBlock_Phoenix_MKDS-1,5-2-5.08_1x02_P5.08mm_Horizontal -> Connector_JST:JST_XH_S2B-XH-A-1_1x02_P2.50mm_Horizontal
- J1: value Conn_01x14_Pin -> Conn_01x16_Pin; footprint Connector_PinHeader_2.54mm:PinHeader_1x14_P2.54mm_Horizontal -> Connector_PinHeader_2.54mm:PinHeader_1x16_P2.54mm_Horizontal
- moved J2 21.0 mm to (167.8, 80.5), turned to 0 degrees
- moved D8 8.39 mm to (114.8, 75.2), turned to 0 degrees
- moved D7 3.96 mm to (122.8, 81.2)
- moved J3 3.42 mm to (148.7, 65.5), turned to 90 degrees
- moved J1 0.38 mm to (113.5, 60.0)
Connections:
- D7 pad 1: +5V -> OUT2U3
- D7 pad 2: OUT1U3 -> GND
- D8 pad 1: +5V -> OUT1U3
- D8 pad 2: OUT2U3 -> GND
- J1 pad 5: SW1U3 -> unconnected-(J1-Pin_5-Pad5)
- J1 pad 6: SW2U3 -> unconnected-(J1-Pin_6-Pad6)
- J2 pad 1: GND -> IN4U2
- J2 pad 2: unconnected-(J2-Pin_2-Pad2) -> IN3U2
- J2 pad 3: +5V -> unconnected-(J2-Pin_3-Pad3)
- J2 pad 4: IN3U2 -> unconnected-(J2-Pin_4-Pad4)
- J2 pad 5: IN4U2 -> +5V
- J2 pad 7: unconnected-(J2-Pin_7-Pad7) -> +5V
- J2 pad 8: +5V -> GND
- J3 pad 1: GND -> IN2U2
- J3 pad 2: unconnected-(J3-Pin_2-Pad2) -> IN1U2
- J3 pad 3: +5V -> unconnected-(J3-Pin_3-Pad3)
- J3 pad 4: IN1U2 -> unconnected-(J3-Pin_4-Pad4)
- J3 pad 5: IN2U2 -> +5V
- J3 pad 7: unconnected-(J3-Pin_7-Pad7) -> +5V
- J3 pad 8: +5V -> GND
- J4 pad 1: +5V -> +12V
- J4 pad 2: +12V -> +5V
- R1 pad 2: GND -> +3.3V
- U3 pad 11: ENBU3 -> +5V
- U3 pad 6: ENAU3 -> +5V
- U3 pad 9: +12V -> +5V
Routing:
- net +3.3V: track 0.00 -> 85.0 mm
- net +12V: track 74.2 -> 11.1 mm
- net SW1U3: track 47.6 -> 0.00 mm
- net SW2U3: track 43.7 -> 0.00 mm
- net ENBU3: track 42.5 -> 0.00 mm
- net OUT2U3: track 43.2 -> 72.4 mm
- net IN4U2: track 8.09 -> 36.9 mm
- net OUT4U3: track 37.7 -> 62.4 mm
- net ENAU3: track 20.1 -> 0.00 mm
- net LIGHT: track 100.0 -> 115.4 mm
- net IN3U3: track 154.7 -> 169.6 mm
- net +5V: track 25.0 -> 37.4 mm, vias 11 -> 15
- net IN3U2: track 27.7 -> 37.2 mm
- net GND: track 26.5 -> 34.1 mm, vias 9 -> 12
- net IN2U2: track 18.8 -> 12.1 mm
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Other:
- board size 70.2 x 54.2 mm -> 78.4 x 54.2 mm
- board text added: "12V"
- board text added: "3.3V"
- board text added: "5V"
- board text added: "GND"
- board text added: "In1H"
- board text added: "In1W"
- board text added: "In2H"
- board text added: "In2W"
- board text added: "In3H"
- board text added: "In3W"
- board text added: "In4H"
- board text added: "In4W"
- board text added: "LT"
- board text added: "NC"
- board text added: "PHTR"
- board text added: "POT"
